File: elec_RPI_Robot_HAT.kicad_sch (KiCad schematic)
At the start: 12 parts, among them J4 THD-20-R

Commit message: [added] datasheets
Parts:
- added H7: MountingHole_Pad, MountingHole:MountingHole_2.7mm_M2.5_ISO7380_Pad_TopBottom, symbol Mechanical:MountingHole_Pad
- J4: footprint Library_Pollen:PinHeader_2x20_P2.54mm_Vertical_with_rasp_HAT -> Library_Pollen:PinHeader_2x20_P2.54mm_Vertical_with_rasp_HAT_zero
Connections:
- net GND: now also H7.1
Other:
- sheet Dynamixel ports: added {GPIO}; removed none
- sheet Sensors ports: added {GPIO}; removed none

Commit message: [update] Thinking about audio.
Parts:
- removed H4, H5, H6, H7: MountingHole_Pad, MountingHole:MountingHole_2.7mm_M2.5_ISO7380_Pad_TopBottom, symbol Mechanical:MountingHole_Pad
- J4: symbol Connector_Generic:Conn_02x20_Odd_Even -> Connector_Generic_MountingPin:Conn_02x20_Odd_Even_MountingPin
Connections:
- net GND: now also J4.MP (MountPin)
Other:
- note added: "Audio part requires: - auto-gain - filters It should at least be 2 inputs + 1 output (could be USB loudspeaker if lacking space). Basic functions: AGC, filters, EQ but no DSP (so echo cancelation, beam forming... will be soft). Output should be 1W (RM is 5W). ICs: WM8960, NAU88C22YG, TLV320AIC3104, TLV320AIC3254, DA7212, TAC5112"
- note added: "Cabled buses: - I2C_ID: HAT identification - I2C0: Cabled GPIOs on the 40-way Header: - GPIO00 - GPIO01 - GPIO02: Stemma/QT - SDA - GPIO03: Stemma/QT - SCL - GPIO04 - GPIO05 - GPIO06 - GPIO07: IMU - Acc_CS - GPIO08: IMU - Gyr_CS - GPIO09: IMU - MISO - GPIO10: IMU - MOSI - GPIO11: IMU - Clk - GPIO12 - GPIO13: Dynamixel - UART_RTS - GPIO14: Dynamixel - UART_Tx - GPIO15: Dynamixel - UART_Rx - GPIO16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"
- note removed: "Cabled buses: - I2C_ID: cam0 and 40Way GPIO Header - I2C0: cam1 and fan controller Cabled GPIOs on the 40-way Header: - GPIO00: used for Cam0 - GPIO01 - GPIO02: Stemma/QT - SDA - GPIO03: Stemma/QT - SCL - GPIO04 - GPIO05 - GPIO06 - GPIO07: IMU - Acc_CS - GPIO08: IMU - Gyr_CS - GPIO09: IMU - MISO - GPIO10: IMU - MOSI - GPIO11: IMU - Clk - GPIO12 - GPIO13: Dynamixel - UART_RTS - GPIO14: Dynamixel -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"
- note removed: "Mounting Holes M2,5"
- moved on the sheet: R8, R9

Commit message: [update] All schematic up.
Parts:
- added C25: 100n, Capacitor_SMD:C_0603_1608Metric, symbol Device:C_Small
- added R10, R11: 10k, Resistor_SMD:R_0402_1005Metric, symbol Device:R_Small
- added U4: CAT24C32HU4, LCSC_parts_lib:TDFN-8_L3.0-W2.0-P0.50-BL-EP, symbol Memory_EEPROM:CAT24C128
Connections:
- net +3V3: now also C25.2, R10.1, R11.1, U4.8 (VCC)
- net GND: now also C25.1, U4.1 (A0), U4.2 (A1), U4.3 (A2), U4.4 (GND)
- net ID_SC: now also R10.2, U4.6 (SCL)
- net ID_SD: now also R11.2, U4.5 (SDA)
- no-connect marks 0 -> 1
Other:
- added sheet Audio (audio.kicad_sch)
- note added: "Cabled GPIOs on the 40-way Header: - GPIO02: Audio + Stemma/QT - SDA - GPIO03: Audio + Stemma/QT - SCL - GPIO04 - GPIO05 - GPIO06 - GPIO07: IMU - Acc_CS - GPIO08: IMU - Gyr_CS - GPIO09: IMU - MISO - GPIO10: IMU - MOSI - GPIO11: IMU - Clk - GPIO12 - GPIO13: Dynamixel - UART_RTS - GPIO14: Dynamixel - UART_Tx - GPIO15: Dynamixel - UART_Rx - GPIO16 - GPIO17 - GPIO18: Audio, PCM Clk - GPIO19: Audio, P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"
- note added: "HAT Identification: I2C add. 0x50 Standard Class HAT+"
- note added: "See: https://github.com/raspberrypi/utils/tree/master/eeptools"
- note added: "ToDo: - HAT+ marking?"
- note removed: "Audio part requires: - auto-gain - filters It should at least be 2 inputs + 1 output (could be USB loudspeaker if lacking space). Basic functions: AGC, filters, EQ but no DSP (so echo cancelation, beam forming... will be soft). Output should be 1W (RM is 5W). ICs: WM8960, NAU88C22YG, TLV320AIC3104, TLV320AIC3254, DA7212, TAC5112"
- note removed: "Cabled buses: - I2C_ID: HAT identification - I2C0: Cabled GPIOs on the 40-way Header: - GPIO00 - GPIO01 - GPIO02: Stemma/QT - SDA - GPIO03: Stemma/QT - SCL - GPIO04 - GPIO05 - GPIO06 - GPIO07: IMU - Acc_CS - GPIO08: IMU - Gyr_CS - GPIO09: IMU - MISO - GPIO10: IMU - MOSI - GPIO11: IMU - Clk - GPIO12 - GPIO13: Dynamixel - UART_RTS - GPIO14: Dynamixel - UART_Tx - GPIO15: Dynamixel - UART_Rx - GPIO16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"
- moved on the sheet: J4, R8, R9

Commit message: [update] Schematic completed.
Parts:
- C25: footprint Capacitor_SMD:C_0603_1608Metric -> Capacitor_SMD:C_0402_1005Metric
Other:
- note added: "Cabled GPIOs on the 40-way Header: - GPIO00/01: HAT identification over I2C (reserved) - GPIO02: IMU + Audio + Stemma/QT - SDA - GPIO03: IMU + Audio + Stemma/QT - SCL - GPIO04: Stemma/QT - SDA - GPIO05: Stemma/QT - SCL - GPIO06 - GPIO07 - GPIO08: Stemma/QT - SDA - GPIO09: Stemma/QT - SCL - GPIO10: Stemma/QT - SDA - GPIO11: Stemma/QT - SCL - GPIO12 - GPIO13: Dynamixel - UART_RTS - GPIO14: Dynamixe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"
- note added: "Cabled buses on Raspberry PIs - PI zero 2W: - I2C0 (pin 27/28 ID_SD/C): HAT identification (reserved) - I2C1 (pin 2/3 SDA/SCL): IMU + Audio + Stemma/QT - PI 4: - same I2C0/1 - I2C4 (pin 8/9 SDA/SCL): Stemma/QT - I2C5 (pin 10/11 SDA/SCL): Stemma/QT - PI 5: - same I2C0/1 - I2C2 (pin 4/5 SDA/SCL): Stemma/QT"
- note removed: "Cabled GPIOs on the 40-way Header: - GPIO02: Audio + Stemma/QT - SDA - GPIO03: Audio + Stemma/QT - SCL - GPIO04 - GPIO05 - GPIO06 - GPIO07: IMU - Acc_CS - GPIO08: IMU - Gyr_CS - GPIO09: IMU - MISO - GPIO10: IMU - MOSI - GPIO11: IMU - Clk - GPIO12 - GPIO13: Dynamixel - UART_RTS - GPIO14: Dynamixel - UART_Tx - GPIO15: Dynamixel - UART_Rx - GPIO16 - GPIO17 - GPIO18: Audio, PCM Clk - GPIO19: Audio, P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"
Changed lines of the file:
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@@
 		)
 	)
+	(text "Cabled buses on Raspberry PIs\n - PI zero 2W:\n     - I2C0 (pin 27/28 ID_SD/C): HAT identification (reserved)\n     - I2C1 (pin 2/3 SDA/SCL): IMU + Audio + Stemma/QT\n - PI 4:\n     - same I2C0/1\n     - I2C4 (pin 8/9 SDA/SCL): Stemma/QT\n     - I2C5 (pin 10/11 SDA/SCL): Stemma/QT\n - PI 5:\n     - same I2C0/1\n     - I2C2 (pin 4/5 SDA/SCL): Stemma/QT"
+		(exclude_from_sim no)
+		(at 181.102 57.912 0)
+		(effects
+			(font
+				(size 2.0066 2.0066)
+			)
+			(justify left bottom)
+		)
+	)
 	(text "EB"
 		(exclude_from_sim no)
@@
 		)
 	)
-	(text "Cabled GPIOs on the 40-way Header:\n - GPIO02: Audio + Stemma/QT - SDA\n - GPIO03: Audio + Stemma/QT - SCL\n - GPIO04\n - GPIO05\n - GPIO06\n - GPIO07: IMU - Acc_CS\n - GPIO08: IMU - Gyr_CS\n - GPIO09: IMU - MISO\n - GPIO10: IMU - MOSI\n - GPIO11: IMU - Clk\n - GPIO12\n - GPIO13: Dynamixel - UART_RTS\n - GPIO14: Dynamixel - UART_Tx\n - GPIO15: Dynamixel - UART_Rx\n - GPIO16\n - GPIO17\n - GPIO18: Audio, PCM Clk\n - GPIO19: Audio, PCM FS\n - GPIO20: Audio, Din\n - GPIO21: Audio, Dout\n - GPIO22\n - GPIO23\n - GPIO24\n - GPIO25\n - GPIO26\n - GPIO27\n - ID_SD/C: HAT identification over I2C\n"
+	(text "Cabled GPIOs on the 40-way Header:\n - GPIO00/01: HAT identification over I2C (reserved)\n - GPIO02: IMU + Audio + Stemma/QT - SDA\n - GPIO03: IMU + Audio + Stemma/QT - SCL\n - GPIO04: Stemma/QT - SDA\n - GPIO05: Stemma/QT - SCL\n - GPIO06\n - GPIO07\n - GPIO08: Stemma/QT - SDA\n - GPIO09: Stemma/QT - SCL\n - GPIO10: Stemma/QT - SDA\n - GPIO11: Stemma/QT - SCL\n - GPIO12\n - GPIO13: Dynamixel - UART_RTS\n - GPIO14: Dynamixel - UART_Tx\n - GPIO15: Dynamixel - UART_Rx\n - GPIO16\n - GPIO17\n - GPIO18: Audio, PCM Clk\n - GPIO19: Audio, PCM FS\n - GPIO20: Audio, Din\n - GPIO21: Audio, Dout\n - GPIO22\n - GPIO23\n - GPIO24\n - GPIO25\n - GPIO26\n - GPIO27\n"
 		(exclude_from_sim no)
 		(at 192.786 154.178 0)
@@
 	(text "See: https://github.com/raspberrypi/utils/tree/master/eeptools"
 		(exclude_from_sim no)
-		(at 67.31 187.96 0)
+		(at 75.946 188.214 0)
 		(effects
 			(font
@@
 			)
 		)
-		(property "Footprint" "Capacitor_SMD:C_0603_1608Metric"
+		(property "Footprint" "Capacitor_SMD:C_0402_1005Metric"
 			(at 63.5 158.75 0)
 			(effects
@@
 	(sheet
 		(at 24.13 80.01)
-		(size 12.7 102.87)
+		(size 12.7 109.22)
 		(exclude_from_sim no)
 		(in_bom yes)
@@
 		)
 		(property "Sheetfile" "power.kicad_sch"
-			(at 24.13 183.4646 0)
+			(at 24.13 189.8146 0)
 			(effects
 				(font

Commit message: [update] Started routing.  Started routing.# Veuillez saisir le message de validation pour vos modifications. Les lignes
Parts:
- removed R8: 0R, Resistor_SMD:R_0402_1005Metric, symbol Device:R_Small
- removed R9: DNP-0R, Resistor_SMD:R_0402_1005Metric, symbol Device:R_Small
Other:
- note removed: "GPIO Voltage select"

Commit message: [update] BU before changing the 40-pin GPIO
Parts:
- J4: LCSC Part (none) -> C2977589
Changed lines of the file:
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@@
+			)
+		)
+		(property "LCSC Part" "C2977589"
+			(at 129.54 107.95 0)
+			(effects
+				(font
+					(size 1.27 1.27)
+				)
+				(hide yes)
 			)
 		)

Commit message: [update] Routing...
Parts:
- J4: footprint Library_Pollen:PinHeader_2x20_P2.54mm_Vertical_with_rasp_HAT_zero -> Library_Pollen:PinHeader_2x20_P2.54mm_Vertical_with_rasp_HAT_zero_SMD_connector
Changed lines of the file:
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@@
 			)
 		)
-		(property "Footprint" "Library_Pollen:PinHeader_2x20_P2.54mm_Vertical_with_rasp_HAT_zero"
+		(property "Footprint" "Library_Pollen:PinHeader_2x20_P2.54mm_Vertical_with_rasp_HAT_zero_SMD_connector"
 			(at 129.54 107.95 0)
 			(effects

Commit message: [update] Fully routed, need DRC!
Parts:
- C25: LCSC Part C85864 -> C307331
Changed lines of the file:
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@@
 			)
 		)
-		(property "LCSC Part" "C85864"
+		(property "LCSC Part" "C307331"
 			(at 63.5 158.75 0)
 			(effects
