File: elec_RPI_Robot_HAT.kicad_sch (KiCad schematic)
At the start: 11 parts, among them J4 THD-20-R, U4 CAT24C32HU4

Commit message: [update] Just figure out the 40-pin GPIO conn. is inverted :-/
Parts:
- H1: value PCB01xyz -> PCB01186
Other:
- note added: "06/03/2026"
- note added: "ASE01187"
- note removed: "23/02/2026"
- note removed: "ASE01xyz"
Changed lines of the file:
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@@
 	(title_block
 		(title "elec RPI Robot HAT")
-		(date "2026-02-23")
+		(date "2026-03-06")
 		(rev "A1")
 		(company "Pollen Robotics/HF")
@@
 		)
 	)
-	(text "ASE01xyz"
+	(text "ASE01187"
 		(exclude_from_sim no)
 		(at 116.84 168.275 0)
@@
 		)
 	)
-	(text "23/02/2026"
+	(text "06/03/2026"
 		(exclude_from_sim no)
 		(at 39.37 44.45 0)
@@
 			)
 		)
-		(property "Value" "PCB01xyz"
+		(property "Value" "PCB01186"
 			(at 116.84 164.465 0)
 			(effects

Commit message: [update] +image
Other:
- note added: ""RPI_Robot_HAT" is a raspberry PI HAT designed for small/medium size robots. It has an IMU, Dynamixel connectors and audio. Its dimensions fits a raspberry PI zero"
- note removed: ""RPI_Robot_HAT" is a raspberry pi HAT designed for small/medium size robots. It has an IMU, Dynamixel connectors and maybe a little bit of audio (fingers crossed)."

Commit message: [update] Release A1, production of 15 boards by JLCPCB
Parts:
- J4: value THD-20-R -> Female Header 2x20 SMD; FT Rotation Offset (none) -> 90; LCSC Part C2977589 -> C2685112
Changed lines of the file:
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@@
 			)
 		)
-		(property "Value" "THD-20-R"
+		(property "Value" "Female Header 2x20 SMD"
 			(at 130.81 81.8896 0)
 			(effects
@@
 					(size 1.27 1.27)
 				)
+				(hide yes)
 			)
 		)
@@
 			)
 		)
-		(property "FT Rotation Offset" ""
+		(property "FT Rotation Offset" "90"
 			(at 129.54 107.95 0)
 			(effects
@@
 			)
 		)
-		(property "LCSC Part" "C2977589"
-			(at 129.54 107.95 0)
-			(effects
+		(property "LCSC Part" "C2685112"
+			(at 129.54 107.95 0)
+			(effects

Commit message: [added] Docs
Other:
- note added: "ToDo: - la position de l'IMU doit être connue - attention la zero est sensible aux coupures de courant - plus de dyn3 (perte de tension au bout de x moteurs) - mettre des jumpers pour transformer des dyn4 en dyn3"
Changed lines of the file:
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@@
+		)
+	)
+	(text "ToDo:\n - la position de l'IMU doit être connue\n - attention la zero est sensible aux coupures de courant\n - plus de dyn3 (perte de tension au bout de x moteurs)\n    - mettre des jumpers pour transformer des dyn4 en dyn3"
+		(exclude_from_sim no)
+		(at 63.246 82.804 0)
+		(effects
+			(font
+				(size 2.007 2.007)
+			)
+			(justify left bottom)
 		)
 	)

Commit message: [update] On-going corrections for B1
Other:
- note added: "ToDo: - oscillator is 180 deg (JLC) - give access to ID_SD/SC via another Qwiic connector - rasp zero 2w is very sensitive to rude shutdowns (SD cards corrupts), a shutdown switch/brown out detector as in RM should be implemented - Dyn3 connectors tends to lose voltage, it would be much better if there are more of them, avoiding long chain of motors on a same bus, or here, turning dyn4 into dyn3 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"
- note added: "[fix] Acc. is at 0x19 I2C address [fix] Soft reset of the audio DAC [fix] Ideal diode [fix] Know position of IMU"
- note removed: "ToDo: - la position de l'IMU doit être connue - attention la zero est sensible aux coupures de courant - plus de dyn3 (perte de tension au bout de x moteurs) - mettre des jumpers pour transformer des dyn4 en dyn3"
Changed lines of the file:
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@@
 		)
 	)
-	(text "ToDo:\n - la position de l'IMU doit être connue\n - attention la zero est sensible aux coupures de courant\n - plus de dyn3 (perte de tension au bout de x moteurs)\n    - mettre des jumpers pour transformer des dyn4 en dyn3"
+	(text "[fix] Acc. is at 0x19 I2C address\n[fix] Soft reset of the audio DAC\n[fix] Ideal diode\n[fix] Know position of IMU"
 		(exclude_from_sim no)
-		(at 63.246 82.804 0)
+		(at 87.884 53.34 0)
+		(effects
+			(font
+				(size 2.0066 2.0066)
+			)
+			(justify left bottom)
+		)
+	)
+	(text "ToDo:\n- oscillator is 180 deg (JLC)\n- give access to ID_SD/SC via another Qwiic connector\n- rasp zero 2w is very sensitive to rude shutdowns (SD cards corrupts), a shutdown switch/brown out detector as in RM should be implemented\n- Dyn3 connectors tends to lose voltage, it would be much better if there are more of them, avoiding long chain of motors on a same bus, or here, turning dyn4 into dyn3 with jumpers\n- 10k/1u between the DAC and the amp?\n- wago connector are not fitted to speaker/mic wires (too thin)\n- 2 mics signals + *2* gnd → wago 4\n- missing DC-cut capacitor behind the dual mic/wago connector\n- move DynDir from IO13 to IO17 so one can use the hard RTS of the rasp\n- IMU should be disconnectable (in order to use an external IMU)."
+		(exclude_from_sim no)
+		(at 62.738 134.62 0)
 		(effects
 			(font
@@
 	(text "ToDo:\n - HAT+ marking?"
 		(exclude_from_sim no)
-		(at 102.616 53.086 0)
+		(at 46.482 61.214 0)
 		(effects
 			(font
@@
 		)
 		(instances
-			(project "elec_forcathon"
+			(project "elec_RPI_Robot_HAT"
 				(path "/bc05f5da-608c-4912-90e4-36b13d989976"
 					(reference "H1")
@@
 		)
 		(instances
-			(project "elec_forcathon"
+			(project "elec_RPI_Robot_HAT"
 				(path "/bc05f5da-608c-4912-90e4-36b13d989976"
 					(reference "FID3")
@@
 		)
 		(instances
-			(project "elec_forcathon"
+			(project "elec_RPI_Robot_HAT"
 				(path "/bc05f5da-608c-4912-90e4-36b13d989976"
 					(reference "FID1")
@@
 		)
 		(instances
-			(project "elec_forcathon"
+			(project "elec_RPI_Robot_HAT"
 				(path "/bc05f5da-608c-4912-90e4-36b13d989976"
 					(reference "FID2")
@@
 		)
 		(instances
-			(project "elec_forcathon"
+			(project "elec_RPI_Robot_HAT"
 				(path "/bc05f5da-608c-4912-90e4-36b13d989976"
 					(reference "H3")
@@
 		)
 		(instances
-			(project ""
+			(project "elec_RPI_Robot_HAT"
 				(path "/bc05f5da-608c-4912-90e4-36b13d989976"
 					(reference "H2")
