File: elec_RPI_Robot_HAT.kicad_sch (KiCad schematic)
At the start: 11 parts, among them J4 Female Header 2x20 SMD, U4 CAT24C32HU4

Commit message: [update] B1-RC1, DRC OK on sch/pcb
Connections:
- net IO_07: no longer names the net of J4.26 (Pin_26)
- net IO_12: no longer names the net of J4.32 (Pin_32)
- net IO_13: no longer names the net of J4.33 (Pin_33)
- net IO_16: no longer names the net of J4.36 (Pin_36)
- net IO_17: no longer names the net of J4.11 (Pin_11)
- net IO_23: no longer names the net of J4.16 (Pin_16)
- net IO_24: no longer names the net of J4.18 (Pin_18)
- net IO_25: no longer names the net of J4.22 (Pin_22)
- net IO_26: no longer names the net of J4.37 (Pin_37)
- net IO_27: no longer names the net of J4.13 (Pin_13)
- no-connect marks 1 -> 11
Other:
- sheet Power ports: added {GPIO}; removed none
- note added: "Cabled GPIOs on the 40-way Header: - GPIO00/01: HAT identification over I2C (reserved) - GPIO02: IMU + Audio + Stemma/QT - SDA - GPIO03: IMU + Audio + Stemma/QT - SCL - GPIO04: Stemma/QT - SDA - GPIO05: Stemma/QT - SCL - GPIO06: Switch off detection - GPIO07 - GPIO08: Stemma/QT - SDA - GPIO09: Stemma/QT - SCL - GPIO10: Stemma/QT - SDA - GPIO11: Stemma/QT - SCL - GPIO12 - GPIO13: - GPIO14: Dynamix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"
- note added: "IO_07"
- note added: "IO_12"
- note added: "IO_13"
- note added: "IO_16"
- note added: "IO_17"
- note added: "IO_23"
- note added: "IO_24"
- note added: "IO_25"
- note added: "IO_26"
- note added: "IO_27"
- note added: "[fix] Acc. is at 0x19 I2C address [fix] Soft reset of the audio DAC [fix] Ideal diode [fix] Know position of IMU [fix] Dynamixel_RTS is now on IO_17 [added] IMU can be disconnected [added] IMU_IT is cabled [added] Access to I2C0 [added] Switch off detection"
- note removed: "Cabled GPIOs on the 40-way Header: - GPIO00/01: HAT identification over I2C (reserved) - GPIO02: IMU + Audio + Stemma/QT - SDA - GPIO03: IMU + Audio + Stemma/QT - SCL - GPIO04: Stemma/QT - SDA - GPIO05: Stemma/QT - SCL - GPIO06 - GPIO07 - GPIO08: Stemma/QT - SDA - GPIO09: Stemma/QT - SCL - GPIO10: Stemma/QT - SDA - GPIO11: Stemma/QT - SCL - GPIO12 - GPIO13: Dynamixel - UART_RTS - GPIO14: Dynamixe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"
- note removed: "ToDo: - oscillator is 180 deg (JLC) - give access to ID_SD/SC via another Qwiic connector - rasp zero 2w is very sensitive to rude shutdowns (SD cards corrupts), a shutdown switch/brown out detector as in RM should be implemented - Dyn3 connectors tends to lose voltage, it would be much better if there are more of them, avoiding long chain of motors on a same bus, or here, turning dyn4 into dyn3 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"
- note removed: "[fix] Acc. is at 0x19 I2C address [fix] Soft reset of the audio DAC [fix] Ideal diode [fix] Know position of IMU"

Commit message: [errors] Missing 3v3 on J8/R38/R39
Other:
- note added: "Cabled buses on Raspberry PIs - PI zero 2W: - I2C0 (pin 27/28 ID_SD/C): HAT identification (reserved) - I2C1 (pin 2/3 SDA/SCL): IMU + Audio + Stemma/QT - PI 4: - same I2C0/1 - I2C3 (pin 7/29 SDA/SCL): Stemma/QT - I2C4 (pin 8/9 SDA/SCL): Stemma/QT - I2C5 (pin 10/11 SDA/SCL): Stemma/QT - PI 5: - same I2C0/1 - I2C2 (pin 4/5 SDA/SCL): Stemma/QT"
- note added: "ToDo: - ERROR: 3v3 is missing on J8, R38/39"
- note removed: "Cabled buses on Raspberry PIs - PI zero 2W: - I2C0 (pin 27/28 ID_SD/C): HAT identification (reserved) - I2C1 (pin 2/3 SDA/SCL): IMU + Audio + Stemma/QT - PI 4: - same I2C0/1 - I2C4 (pin 8/9 SDA/SCL): Stemma/QT - I2C5 (pin 10/11 SDA/SCL): Stemma/QT - PI 5: - same I2C0/1 - I2C2 (pin 4/5 SDA/SCL): Stemma/QT"
Changed lines of the file:
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@@
 		)
 	)
-	(text "Cabled buses on Raspberry PIs\n - PI zero 2W:\n     - I2C0 (pin 27/28 ID_SD/C): HAT identification (reserved)\n     - I2C1 (pin 2/3 SDA/SCL): IMU + Audio + Stemma/QT\n - PI 4:\n     - same I2C0/1\n     - I2C4 (pin 8/9 SDA/SCL): Stemma/QT\n     - I2C5 (pin 10/11 SDA/SCL): Stemma/QT\n - PI 5:\n     - same I2C0/1\n     - I2C2 (pin 4/5 SDA/SCL): Stemma/QT"
+	(text "Cabled buses on Raspberry PIs\n - PI zero 2W:\n     - I2C0 (pin 27/28 ID_SD/C): HAT identification (reserved)\n     - I2C1 (pin 2/3 SDA/SCL): IMU + Audio + Stemma/QT\n - PI 4:\n     - same I2C0/1\n     - I2C3 (pin 7/29 SDA/SCL): Stemma/QT\n     - I2C4 (pin 8/9 SDA/SCL): Stemma/QT\n     - I2C5 (pin 10/11 SDA/SCL): Stemma/QT\n - PI 5:\n     - same I2C0/1\n     - I2C2 (pin 4/5 SDA/SCL): Stemma/QT"
 		(exclude_from_sim no)
 		(at 181.102 57.912 0)
@@
 		)
 	)
+	(text "ToDo:\n - ERROR: 3v3 is missing on J8, R38/39"
+		(exclude_from_sim no)
+		(at 51.054 111.252 0)
+		(effects
+			(font
+				(size 2.0066 2.0066)
+			)
+			(justify left bottom)
+		)
+	)

Commit message: [update] JLC order
Parts:
- C25: value 100n -> DNP-100n; LCSC Part C307331 -> (none); now not fitted
- R10, R11: value 10k -> DNP-10k; LCSC Part C25744 -> (none); now not fitted
- U4: value CAT24C32HU4 -> DNP-CAT24C32HU4; LCSC Part C233772 -> (none); now not fitted
Other:
- note added: "ERROR on B1: - MOS transistor of the ideal diode is reversed (source/drain). It runs as is but it does not protect the DCDC when USB-powered"
- note added: "[fixed] Acc. is at 0x19 I2C address [fixed] Soft reset of the audio DAC [fixed] Ideal diode [fixed] Know position of IMU [update] Dynamixel_dir is based on Tx [added] IMU can be disconnected [added] IMU_IT is cabled [added] Access to I2C0 [added] Switch off detection"
- note removed: "[fix] Acc. is at 0x19 I2C address [fix] Soft reset of the audio DAC [fix] Ideal diode [fix] Know position of IMU [fix] Dynamixel_RTS is now on IO_17 [added] IMU can be disconnected [added] IMU_IT is cabled [added] Access to I2C0 [added] Switch off detection"
Changed lines of the file:
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@@
 		)
 	)
-	(text "[fix] Acc. is at 0x19 I2C address\n[fix] Soft reset of the audio DAC\n[fix] Ideal diode\n[fix] Know position of IMU\n[fix] Dynamixel_RTS is now on IO_17\n[added] IMU can be disconnected\n[added] IMU_IT is cabled\n[added] Access to I2C0\n[added] Switch off detection"
+	(text "[fixed] Acc. is at 0x19 I2C address\n[fixed] Soft reset of the audio DAC\n[fixed] Ideal diode\n[fixed] Know position of IMU\n[update] Dynamixel_dir is based on Tx\n[added] IMU can be disconnected\n[added] IMU_IT is cabled\n[added] Access to I2C0\n[added] Switch off detection"
 		(exclude_from_sim no)
 		(at 93.218 75.438 0)
@@
 		)
 	)
+	(text "ERROR on B1:\n - MOS transistor of the ideal diode is reversed (source/drain). \n   It runs as is but it does not protect the DCDC when USB-powered"
+		(exclude_from_sim no)
+		(at 57.658 120.396 0)
+		(effects
+			(font
+				(size 2.0066 2.0066)
+			)
+			(justify left bottom)
+		)
+	)
 	(text "EB"
 		(exclude_from_sim no)
@@
 		(in_bom yes)
 		(on_board yes)
-		(dnp no)
+		(dnp yes)
 		(property "Reference" "R10"
 			(at 73.152 160.782 0)
@@
 			)
 		)
-		(property "Value" "10k"
-			(at 73.406 157.48 0)
+		(property "Value" "DNP-10k"
+			(at 76.454 155.956 0)
 			(effects
 				(font
@@
 			)
 		)
-		(property "LCSC Part" "C25744"
+		(property "LCSC Part" ""
 			(at 77.47 160.02 90)
 			(effects
@@
 		(in_bom yes)
 		(on_board yes)
-		(dnp no)
+		(dnp yes)
 		(property "Reference" "U4"
 			(at 50.8 166.37 0)
@@
 			)
 		)
-		(property "Value" "CAT24C32HU4"
+		(property "Value" "DNP-CAT24C32HU4"
 			(at 70.104 179.324 0)
 			(effects
@@
 			)
 		)
-		(property "LCSC Part" "C233772"
+		(property "LCSC Part" ""
 			(at 55.88 172.72 0)
 			(effects
@@
 		(in_bom yes)
 		(on_board yes)
-		(dnp no)
+		(dnp yes)
 		(property "Reference" "C25"
 			(at 68.072 156.464 0)
@@
 			)
 		)
-		(property "Value" "100n"
+		(property "Value" "DNP-100n"
 			(at 69.342 160.274 0)
 			(effects
@@
 			)
 		)
-		(property "LCSC Part" "C307331"
+		(property "LCSC Part" ""
 			(at 63.5 158.75 0)
 			(effects
@@
 		(in_bom yes)
 		(on_board yes)
-		(dnp no)
+		(dnp yes)
 		(property "Reference" "R11"
 			(at 73.152 162.56 0)
@@
 			)
 		)
-		(property "Value" "10k"
+		(property "Value" "DNP-10k"
 			(at 77.978 161.544 0)
 			(effects
@@
 			)
 		)
-		(property "LCSC Part" "C25744"
+		(property "LCSC Part" ""
 			(at 81.28 160.02 90)
 			(effects

Commit message: [release] B1 (has been produced qtty 125 by JLCPCB)
Parts:
- removed C25: DNP-100n, Capacitor_SMD:C_0402_1005Metric, symbol Device:C_Small
- removed J4: Female Header 2x20 SMD, Library_Pollen:PinHeader_2x20_P2.54mm_Vertical_with_rasp_HAT_zero_SMD_connector, symbol Connector_Generic_MountingPin:Conn_02x20_Odd_Even_MountingPin
- removed R10, R11: DNP-10k, Resistor_SMD:R_0402_1005Metric, symbol Device:R_Small
- removed U4: DNP-CAT24C32HU4, LCSC_parts_lib:TDFN-8_L3.0-W2.0-P0.50-BL-EP, symbol Memory_EEPROM:CAT24C128
Connections:
- no-connect marks 11 -> 0
Other:
- removed sheet Audio
- removed sheet Dynamixel
- removed sheet Power
- removed sheet Sensors
- added sheet Schematic (main.kicad_sch)
- note added: "06/05/2026"
- note added: "B1"
- note added: "ToDo: - HAT+ marking? - ERROR: MOS transistor of the ideal diode is reversed (source/drain). It runs as is but it does not protect the DCDC when USB-powered - ERROR: 3v3 is missing on J8, R38/39"
- note removed: "40Way GPIO Header"
- note removed: "ERROR on B1: - MOS transistor of the ideal diode is reversed (source/drain). It runs as is but it does not protect the DCDC when USB-powered"
- note removed: "HAT Identification: I2C add. 0x50 Standard Class HAT+"
- note removed: "IO_07"
- note removed: "IO_12"
- note removed: "IO_13"
- note removed: "IO_16"
- note removed: "IO_17"
- note removed: "IO_23"
- note removed: "IO_24"
- note removed: "IO_25"
- note removed: "IO_26"
- note removed: "IO_27"
- note removed: "See: https://github.com/raspberrypi/utils/tree/master/eeptools"
- note removed: "ToDo: - ERROR: 3v3 is missing on J8, R38/39"
- note removed: "ToDo: - HAT+ marking?"
- company: Pollen Robotics/HF -> Pollen Robotics / Hugging Face
