File: sensors.kicad_sch (KiCad schematic)
At the start: 6 parts, among them J18 JST SH, U10 BMI088

Commit message: [update] All schematic up.
Other:
- note added: "IMU"
- moved on the sheet: C23, C24, J18, R36, R37, U10

Commit message: [update] Schematic completed.
Parts:
- removed J18: JST SH, Connector_JST:JST_SH_BM04B-SRSS-TB_1x04-1MP_P1.00mm_Vertical, symbol Connector_Generic_MountingPin:Conn_01x04_MountingPin
- removed U10: BMI088, Library_Pollen:BMI088, symbol Library_Pollen:BMI088
- added J5, J6, J7, J8: JST SH, Connector_JST:JST_SH_BM04B-SRSS-TB_1x04-1MP_P1.00mm_Vertical, symbol Connector_Generic_MountingPin:Conn_01x04_MountingPin
- added R12, R13, R20, R21, R34, R35, R38, R39: 10k, Resistor_SMD:R_0402_1005Metric, symbol Device:R_Small
- added R14, R15, R16, R19, R23: 0R, Resistor_SMD:R_0402_1005Metric, symbol Device:R_Small
- added R17, R18, R22: DNP-0R, Resistor_SMD:R_0402_1005Metric, symbol Device:R_Small
- added TP4: TestPoint, TestPoint:TestPoint_THTPad_D2.5mm_Drill1.2mm, symbol Connector:TestPoint
- added U11: BMI088, Package_LGA:Bosch_LGA-16_4.5x3mm_P0.5mm_LayoutBorder7x1y_ClockwisePinNumbering, symbol Sensor_Motion:BMI088
- R36: value 0R -> DNP-0R; now not fitted
- R37: value DNP-0R -> 0R; now fitted
Connections:
- net +3V3: now also R37.1, R16.1, R19.1, R23.1, U11.11 (VDDIO), U11.3 (VDD), U11.7 (PS); no longer R36.1
- net +5V: now also R36.1, R17.1, R18.1, R22.1; no longer R37.1
- net GND: now also J5.1 (Pin_1), J5.MP (MountPin), J6.1 (Pin_1), J6.MP (MountPin), J7.1 (Pin_1), J7.MP (MountPin), J8.1 (Pin_1), J8.MP (MountPin), R14.1, R15.1, U11.2 (GNDA), U11.4 (GNDA), U11.6 (GNDIO)
- net IO_02: now also J5.3 (Pin_3), R12.2, U11.9 (SDI/SDA)
- net IO_03: now also J5.4 (Pin_4), R13.2, U11.8 (SCK/SCL)
- net IO_08: now also J7.3 (Pin_3), R34.2
- net IO_09: now also J7.4 (Pin_4), R35.2
- net IO_10: now also J8.3 (Pin_3), R38.2
- net IO_11: now also J8.4 (Pin_4), R39.2
- net at R36.2, R37.2: now also J8.2 (Pin_2), R38.1, R39.1
- new net: J7.2 (Pin_2), R22.2, R23.2, R34.1, R35.1
- new net: J6.2 (Pin_2), R18.2, R19.2, R20.1, R21.1
- new net: J5.2 (Pin_2), R12.1, R13.1, R16.2, R17.2
- new net: R15.2, U11.10 (SDO2)
- new net: R14.2, U11.15 (SDO1)
- new net: TP4.1, U11.16 (INT1)
- new net IO_04: J6.3 (Pin_3), R20.2
- new net IO_05: J6.4 (Pin_4), R21.2
- no-connect marks 4 -> 5
Other:
- note removed: "Acc_CS"
- note removed: "Gyr_CS"
- note removed: "IMU_MISO"
- note removed: "IMU_MOSI"
- note removed: "IMU_Sck"
- moved on the sheet: C23, C24

Commit message: [update] BU before changing the 40-pin GPIO
Parts:
- TP4: footprint TestPoint:TestPoint_THTPad_D2.5mm_Drill1.2mm -> TestPoint:TestPoint_Loop_D2.50mm_Drill1.0mm_LowProfile
Changed lines of the file:
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@@
 			)
 		)
-		(property "Footprint" "TestPoint:TestPoint_THTPad_D2.5mm_Drill1.2mm"
+		(property "Footprint" "TestPoint:TestPoint_Loop_D2.50mm_Drill1.0mm_LowProfile"
 			(at 245.11 99.06 0)
 			(effects

Commit message: [update] Just figure out the 40-pin GPIO conn. is inverted :-/
Parts:
- renumbered TP4 to IMU_IT1
Changed lines of the file:
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@@
 		(dnp no)
 		(fields_autoplaced yes)
-		(property "Reference" "TP4"
+		(property "Reference" "IMU_IT1"
 			(at 250.19 93.9799 90)
 			(effects
@@
 			(project ""
 				(path "/bc05f5da-608c-4912-90e4-36b13d989976/51aae2c5-2ebf-4088-ad60-315661d0a581"
-					(reference "TP4")
+					(reference "IMU_IT1")
 					(unit 1)
 				)

Commit message: [update] Release A1, production of 15 boards by JLCPCB
Parts:
- J5, J6, J7, J8: LCSC Part C51940130 -> C160390
- U11: FT Rotation Offset -90 -> 180
- renumbered IMU_IT1 to TP1
Changed lines of the file:
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@@
 			)
 		)
-		(property "LCSC Part" "C51940130"
+		(property "LCSC Part" "C160390"
 			(at 127 105.41 0)
 			(effects
@@
 			)
 		)
-		(property "FT Rotation Offset" "-90"
+		(property "FT Rotation Offset" "180"
 			(at 231.14 101.6 0)
 			(effects
@@
 			)
 		)
-		(property "LCSC Part" "C51940130"
+		(property "LCSC Part" "C160390"
 			(at 127 72.39 0)
 			(effects
@@
 			)
 		)
-		(property "LCSC Part" "C51940130"
+		(property "LCSC Part" "C160390"
 			(at 127 171.45 0)
 			(effects
@@
 		(dnp no)
 		(fields_autoplaced yes)
-		(property "Reference" "IMU_IT1"
+		(property "Reference" "TP1"
 			(at 250.19 93.9799 90)
 			(effects
@@
 			(project ""
 				(path "/bc05f5da-608c-4912-90e4-36b13d989976/51aae2c5-2ebf-4088-ad60-315661d0a581"
-					(reference "IMU_IT1")
+					(reference "TP1")
 					(unit 1)
 				)
@@
 			)
 		)
-		(property "LCSC Part" "C51940130"
+		(property "LCSC Part" "C160390"
 			(at 127 137.16 0)
 			(effects

Commit message: [update] On-going corrections for B1
Parts:
- TP1: footprint TestPoint:TestPoint_Loop_D2.50mm_Drill1.0mm_LowProfile -> TestPoint:TestPoint_THTPad_D1.0mm_Drill0.5mm
Connections:
- net +3V3: now also R14.1
- net GND: no longer R14.1
Other:
- note added: "I2C add.: - acc.: 0x19 - gyr.: 0x68"
Changed lines of the file:
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@@
 		)
 	)
+	(text "I2C add.:\n - acc.: 0x19\n - gyr.: 0x68"
+		(exclude_from_sim no)
+		(at 229.616 135.636 0)
+		(effects
+			(font
+				(size 2 2)
+				(thickness 0.4)
+				(bold yes)
+			)
+		)
+	)
 	(text "SDA"
 		(exclude_from_sim no)
@@
 	)
 	(junction
-		(at 204.47 106.68)
-		(diameter 0)
-		(color 0 0 0 0)
-	)
-	(junction
 		(at 106.68 162.56)
 		(diameter 0)
@@
 	(wire
 		(pts
+			(xy 200.66 104.14) (xy 209.55 104.14)
+		)
+		(stroke
+			(width 0)
+			(type default)
+		)
+	)
+	(wire
+		(pts
 			(xy 214.63 106.68) (xy 218.44 106.68)
 		)
@@
 	(wire
 		(pts
-			(xy 209.55 104.14) (xy 204.47 104.14)
-		)
-		(stroke
-			(width 0)
-			(type default)
-		)
-	)
-	(wire
-		(pts
 			(xy 90.17 93.98) (xy 90.17 90.17)
 		)
@@
 	(wire
 		(pts
-			(xy 204.47 104.14) (xy 204.47 106.68)
-		)
-		(stroke
-			(width 0)
-			(type default)
-		)
-	)
-	(wire
-		(pts
 			(xy 115.57 63.5) (xy 115.57 72.39)
 		)
@@
 	)
 	(symbol
+		(lib_id "power:+3V3")
+		(at 200.66 104.14 90)
+		(unit 1)
+		(exclude_from_sim no)
+		(in_bom yes)
+		(on_board yes)
+		(dnp no)
+		(fields_autoplaced yes)
+		(property "Reference" "#PWR029"
+			(at 204.47 104.14 0)
+			(effects
+				(font
+					(size 1.27 1.27)
+				)
+				(hide yes)
+			)
+		)
+		(property "Value" "+3V3"
+			(at 196.85 104.1399 90)
+			(effects
+				(font
+					(size 1.27 1.27)
+				)
+				(justify left)
+			)
+		)
+		(property "Footprint" ""
+			(at 200.66 104.14 0)
+			(effects
+				(font
+					(size 1.27 1.27)
+				)
+				(hide yes)
+			)
+		)
+		(property "Datasheet" ""
+			(at 200.66 104.14 0)
+			(effects
+				(font
+					(size 1.27 1.27)
+				)
+				(hide yes)
+			)
+		)
+		(property "Description" "Power symbol creates a global label with name \"+3V3\""
+			(at 200.66 104.14 0)
+			(effects
+				(font
+					(size 1.27 1.27)
+				)
+				(hide yes)
+			)
+		)
+		(pin "1"
+		)
+		(instances
+			(project "elec_RPI_Robot_HAT"
+				(path "/bc05f5da-608c-4912-90e4-36b13d989976/51aae2c5-2ebf-4088-ad60-315661d0a581"
+					(reference "#PWR029")
+					(unit 1)
+				)
+			)
+		)
+	)
+	(symbol
 		(lib_id "power:GND")
 		(at 204.47 118.11 0)
@@
 		)
 		(instances
-			(project ""
+			(project "elec_RPI_Robot_HAT"
 				(path "/bc05f5da-608c-4912-90e4-36b13d989976/51aae2c5-2ebf-4088-ad60-315661d0a581"
 					(reference "U11")
@@
 		)
 		(instances
-			(project "elec_RPI_Robot_Board_CMx_Carrier"
+			(project "elec_RPI_Robot_HAT"
 				(path "/bc05f5da-608c-4912-90e4-36b13d989976/51aae2c5-2ebf-4088-ad60-315661d0a581"
 					(reference "C24")
@@
 		)
 		(instances
-			(project "elec_RPI_Robot_Board_CMx_Carrier"
+			(project "elec_RPI_Robot_HAT"
 				(path "/bc05f5da-608c-4912-90e4-36b13d989976/51aae2c5-2ebf-4088-ad60-315661d0a581"
 					(reference "#PWR0112")
@@
 		)
 		(instances
-			(project "elec_RPI_Robot_Board_CMx_Carrier"
+			(project "elec_RPI_Robot_HAT"
 				(path "/bc05f5da-608c-4912-90e4-36b13d989976/51aae2c5-2ebf-4088-ad60-315661d0a581"
 					(reference "C23")
@@
 			)
 		)
-		(property "Footprint" "TestPoint:TestPoint_Loop_D2.50mm_Drill1.0mm_LowProfile"
+		(property "Footprint" "TestPoint:TestPoint_THTPad_D1.0mm_Drill0.5mm"
 			(at 245.11 99.06 0)
 			(effects
@@
 		)
 		(instances
-			(project ""
+			(project "elec_RPI_Robot_HAT"
 				(path "/bc05f5da-608c-4912-90e4-36b13d989976/51aae2c5-2ebf-4088-ad60-315661d0a581"
 					(reference "TP1")

Commit message: [update] B1-RC1, DRC OK on sch/pcb
Parts:
- removed R22, R36: DNP-0R, Resistor_SMD:R_0402_1005Metric, symbol Device:R_Small
- removed R23, R37: 0R, Resistor_SMD:R_0402_1005Metric, symbol Device:R_Small
- removed TP1: TestPoint, TestPoint:TestPoint_THTPad_D1.0mm_Drill0.5mm, symbol Connector:TestPoint
- added R25, R9: 0R, Resistor_SMD:R_0402_1005Metric, symbol Device:R_Small
- R17: value DNP-0R -> 0R; now fitted
- R19: value 0R -> DNP-0R; now not fitted
Connections:
- net +3V3: now also J5.2 (Pin_2), J6.2 (Pin_2), J7.2 (Pin_2), R12.1, R13.1, R20.1, R21.1, R34.1, R35.1, R9.2; no longer C23.1, C24.2, R16.1, R19.1, U11.11 (VDDIO), U11.3 (VDD)
- net IO_04: now also R18.1; no longer J6.3 (Pin_3), R20.2
- net IO_05: now also R19.1; no longer J6.4 (Pin_4), R21.2
- net at U11.16 (INT1): now also R25.2
- net +5V renamed ID_SD
- net ID_SD: no longer R18.1
- new net: J6.4 (Pin_4), R16.2, R19.2, R21.2
- new net: J6.3 (Pin_3), R17.2, R18.2, R20.2
- new net: C23.1, C24.2, R9.1, U11.11 (VDDIO), U11.3 (VDD)
- new net ID_SC: R16.1
- new net IO_22: R25.1
Other:
- moved on the sheet: C23, C24, J5, J6, J7, J8, R12, R13, R14, R15, R20, R21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
