File: main.kicad_sch (KiCad schematic)
At the start: 23 parts, among them J5 JST SH, J6 JST SH, J7 JST SH, J8 JST SH, U11 BMI088

Commit message: [release] B1 (has been produced qtty 125 by JLCPCB)
Parts:
- removed C23, C24: 100n 6V3, Capacitor_SMD:C_0402_1005Metric, symbol Device:C_Small
- removed J5, J6, J7, J8: JST SH, Connector_JST:JST_SH_BM04B-SRSS-TB_1x04-1MP_P1.00mm_Vertical, symbol Connector_Generic_MountingPin:Conn_01x04_MountingPin
- removed R12, R13, R20, R21, R34, R35, R38, R39: 10k, Resistor_SMD:R_0402_1005Metric, symbol Device:R_Small
- removed R14, R15, R16, R17, R25, R9: 0R, Resistor_SMD:R_0402_1005Metric, symbol Device:R_Small
- removed R18, R19: DNP-0R, Resistor_SMD:R_0402_1005Metric, symbol Device:R_Small
- removed U11: BMI088, Package_LGA:Bosch_LGA-16_4.5x3mm_P0.5mm_LayoutBorder7x1y_ClockwisePinNumbering, symbol Sensor_Motion:BMI088
- added C25: DNP-100n, Capacitor_SMD:C_0402_1005Metric, symbol Device:C_Small
- added J4: Female Header 2x20 SMD, Library_Pollen:PinHeader_2x20_P2.54mm_Vertical_with_rasp_HAT_zero_SMD_connector, symbol Connector_Generic_MountingPin:Conn_02x20_Odd_Even_MountingPin
- added R10, R11: DNP-10k, Resistor_SMD:R_0402_1005Metric, symbol Device:R_Small
- added U4: DNP-CAT24C32HU4, LCSC_parts_lib:TDFN-8_L3.0-W2.0-P0.50-BL-EP, symbol Memory_EEPROM:CAT24C128
Connections:
- net +3V3: now also C25.2, J4.1 (Pin_1), J4.17 (Pin_17), R10.1, R11.1, U4.8 (VCC)
- net GND: now also C25.1, J4.14 (Pin_14), J4.20 (Pin_20), J4.25 (Pin_25), J4.30 (Pin_30), J4.34 (Pin_34), J4.39 (Pin_39), J4.6 (Pin_6), J4.9 (Pin_9), J4.MP (MountPin), U4.1 (A0), U4.2 (A1), U4.3 (A2), U4.4 (GND)
- net ID_SC: now also J4.28 (Pin_28), R10.2, U4.6 (SCL)
- net ID_SD: now also J4.27 (Pin_27), R11.2, U4.5 (SDA)
- net IO_02: now also J4.3 (Pin_3)
- net IO_03: now also J4.5 (Pin_5)
- net IO_04: now also J4.7 (Pin_7)
- net IO_05: now also J4.29 (Pin_29)
- net IO_08: now also J4.24 (Pin_24)
- net IO_09: now also J4.21 (Pin_21)
- net IO_10: now also J4.19 (Pin_19)
- net IO_11: now also J4.23 (Pin_23)
- net IO_22: now also J4.15 (Pin_15)
- new net +5V: J4.2 (Pin_2), J4.4 (Pin_4)
- new net IO_06: J4.31 (Pin_31)
- new net IO_14: J4.8 (Pin_8)
- new net IO_15: J4.10 (Pin_10)
- new net IO_18: J4.12 (Pin_12)
- new net IO_19: J4.35 (Pin_35)
- new net IO_20: J4.38 (Pin_38)
- new net IO_21: J4.40 (Pin_40)
- no-connect marks 5 -> 11
Other:
- added sheet Audio (audio.kicad_sch)
- added sheet Dynamixel (dynamixel.kicad_sch)
- added sheet Power (power.kicad_sch)
- added sheet Sensors (sensors.kicad_sch)
- note added: "40Way GPIO Header"
- note added: "HAT Identification: I2C add. 0x50 Standard Class HAT+"
- note added: "IO_07"
- note added: "IO_12"
- note added: "IO_13"
- note added: "IO_16"
- note added: "IO_17"
- note added: "IO_23"
- note added: "IO_24"
- note added: "IO_25"
- note added: "IO_26"
- note added: "IO_27"
- note added: "See: https://github.com/raspberrypi/utils/tree/master/eeptools"
- note removed: "3V3 Default"
- note removed: "I2C add.: - acc.: 0x19 - gyr.: 0x68"
- note removed: "IMU"
- note removed: "SCL"
- note removed: "SDA"
- note removed: "STEMMA QT 1mm"
