File: main.kicad_sch (KiCad schematic)
At the start: 5 parts, among them J4 Female Header 2x20 SMD, U4 DNP-CAT24C32HU4

Commit message: [update] post-Claude corrections
Other:
- note added: "HAT Identification: I2C add. 0x50"
- note removed: "HAT Identification: I2C add. 0x50 Standard Class HAT+"
Changed lines of the file:
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@@
 		)
 	)
-	(text "HAT Identification:\n  I2C add. 0x50\n  Standard Class HAT+"
+	(text "HAT Identification:\n  I2C add. 0x50"
 		(exclude_from_sim no)
 		(at 121.92 151.638 0)
