File: power.kicad_sch (KiCad schematic)
At the start: 14 parts, among them Q2 SI2312CDS-T1-GE3, U10 LM5050-1, U9 AP63205

Commit message: [update] Release C1 (for Grabette), now qtty 20 @JLCPCB
Connections:
- net +5V: now also Q2.3 (D); no longer Q2.2 (S)
- net at C21.1, C22.1, D1.3 (K)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: now also Q2.2 (S); no longer Q2.3 (D)
Other:
- moved on the sheet: Q2
Changed lines of the file:
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@@
 	(symbol
 		(lib_id "Transistor_FET_Other:Q_NMOS_Depletion_GSD")
-		(at 198.12 74.93 90)
+		(at 198.12 74.93 270)
+		(mirror x)
 		(unit 1)
 		(exclude_from_sim no)
@@
 		(on_board yes)
 		(dnp no)
-		(fields_autoplaced yes)
 		(property "Reference" "Q2"
 			(at 198.12 68.58 90)

Commit message: [update] JLC-ready, time for Claude review
Parts:
- Q2: value SI2312CDS-T1-GE3 -> N-Channel 5A; LCSC Part C142518 -> C22469448
Changed lines of the file:
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@@
 			)
 		)
-		(property "Value" "SI2312CDS-T1-GE3"
+		(property "Value" "N-Channel 5A"
 			(at 198.12 68.58 90)
 			(effects
@@
 			)
 		)
-		(property "LCSC Part" "C142518"
+		(property "LCSC Part" "C22469448"
 			(at 198.12 74.93 90)
 			(effects

Commit message: [update] post-Claude corrections
Parts:
- added C45: 10u 35V, Capacitor_SMD:C_0805_2012Metric, symbol Device:C_Small
- C21, C22: symbol Device:C_Polarized_Small -> Device:C_Small
Connections:
- net +BATT: now also C45.1
- net GND: now also C45.2
Other:
- moved on the sheet: C19
